File: coprocessor-psu.kicad_pcb (KiCad board)
At the start: 2 copper layers, 15 parts, among them Q1 Q_NMOS_SGD, U1 LM3488

Commit message: some more details
Parts:
- added ?: , , F.Cu at (156.2, 119.0)
- added ?: , , F.Cu at (109.0, 119.0)
- added ?: , , F.Cu at (109.0, 92.8)
- added REF**: MountingHole_3.2mm_M3_Pad, MountingHole:MountingHole_3.2mm_M3_Pad, F.Cu at (156.2, 92.8)
- moved L1 53.8 mm to (123.2, 95.8)
- moved C1 51.6 mm to (115.8, 110.8), turned to -90 degrees
- moved C4 49.4 mm to (155.5, 107.5), turned to -90 degrees
- moved C3 47.6 mm to (146.5, 107.5)
- moved R3 36.9 mm to (137.0, 111.2)
- moved C5 36.6 mm to (124.5, 121.8)
- moved C6 36.6 mm to (126.5, 121.8)
- moved R2 36.6 mm to (126.5, 125.2)
- moved R4 36.6 mm to (128.5, 121.8)
- moved R5 36.6 mm to (130.5, 121.8)
- moved Q1 36.5 mm to (137.8, 105.5)
- moved U1 36.1 mm to (146.0, 120.2)
- moved C2 36.1 mm to (125.0, 110.8)
- moved D1 35.9 mm to (143.0, 95.8)
- moved R1 33.8 mm to (138.5, 121.8)
Changed lines of the file:
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@@
   (setup
     (pad_to_mask_clearance 0)
+    (aux_axis_origin 100 125)
+    (grid_origin 100 125)
     (pcbplotparams
       (layerselection 0x00010fc_ffffffff)
@@
   (net 10 "Net-(R4-Pad2)")
   (footprint "Package_SO:VSSOP-8_3.0x3.0mm_P0.65mm" (layer "F.Cu")
-    (at 157.5 86)
+    (at 146 120.25)
     (descr "VSSOP-8 3.0 x 3.0, http://www.ti.com/lit/ds/symlink/lm75b.pdf")
     (tags "VSSOP-8 3.0 x 3.0")
@@
     )
   )
+  (footprint "" locked (layer "F.Cu")
+    (at 156.2 119)
+    (fp_text reference "" (at 0 0) (layer "F.SilkS")
+      (effects (font (size 1.27 1.27) (thickness 0.15)))
+    )
+    (fp_text value "" (at 0 0) (layer "F.SilkS")
+      (effects (font (size 1.27 1.27) (thickness 0.15)))
+    )
+    (pad "1" thru_hole circle locked (at 0 0) (size 6.4 6.4) (drill 3.2) (layers F&B.Cu *.Mask))
+  )
   (footprint "Resistor_SMD:R_0805_2012Metric" (layer "F.Cu")
-    (at 157.75 94)
+    (at 138.5 121.75)
     (descr "Resistor SMD 0805 (2012 Metric), square (rectangular) end terminal, IPC_7351 nominal, (Body size source: IPC-SM-782 page 72, https://www.pcb-3d.com/wordpress/wp-content/uploads/ipc-sm-782a_amendment_1_and_2.pdf), generated with kicad-footprint-generator")
     (tags "resistor")
@@
   )
   (footprint "Capacitor_SMD:C_0805_2012Metric" (layer "F.Cu")
-    (at 145.5 91.75 90)
+    (at 124.5 121.75 90)
     (descr "Capacitor SMD 0805 (2012 Metric), square (rectangular) end terminal, IPC_7351 nominal, (Body size source: IPC-SM-782 page 76, https://www.pcb-3d.com/wordpress/wp-content/uploads/ipc-sm-782a_amendment_1_and_2.pdf, https://docs.google.com/spreadsheets/d/1BsfQQcO9C6DZCsRaXUlFlo91Tg2WpOkGARC1WS5S8t0/edit?usp=sharing), generated with kicad-footprint-generator")
     (tags "capacitor")
@@
   )
   (footprint "Capacitor_SMD:C_0805_2012Metric" (layer "F.Cu")
-    (at 147.5 91.75 90)
+    (at 126.5 121.75 90)
     (descr "Capacitor SMD 0805 (2012 Metric), square (rectangular) end terminal, IPC_7351 nominal, (Body size source: IPC-SM-782 page 76, https://www.pcb-3d.com/wordpress/wp-content/uploads/ipc-sm-782a_amendment_1_and_2.pdf, https://docs.google.com/spreadsheets/d/1BsfQQcO9C6DZCsRaXUlFlo91Tg2WpOkGARC1WS5S8t0/edit?usp=sharing), generated with kicad-footprint-generator")
     (tags "capacitor")
@@
   )
   (footprint "Resistor_SMD:R_0805_2012Metric" (layer "F.Cu")
-    (at 149.5 91.75 90)
+    (at 128.5 121.75 90)
     (descr "Resistor SMD 0805 (2012 Metric), square (rectangular) end terminal, IPC_7351 nominal, (Body size source: IPC-SM-782 page 72, https://www.pcb-3d.com/wordpress/wp-content/uploads/ipc-sm-782a_amendment_1_and_2.pdf), generated with kicad-footprint-generator")
     (tags "resistor")
@@
   )
   (footprint "Library:XAL1580" (layer "F.Cu")
-    (at 160.25 56.75)
+    (at 123.25 95.75)
     (property "Sheetfile" "coprocessor-psu.kicad_sch")
     (property "Sheetname" "")
@@
   )
   (footprint "Package_TO_SOT_SMD:TO-263-2" (layer "F.Cu")
-    (at 171.75 74.25)
+    (at 143 95.75)
     (descr "TO-263 / D2PAK / DDPAK SMD package, http://www.infineon.com/cms/en/product/packages/PG-TO263/PG-TO263-3-1/")
     (tags "D2PAK DDPAK TO-263 D2PAK-3 TO-263-3 SOT-404")
@@
     )
   )
+  (footprint "" locked (layer "F.Cu")
+    (at 109 119)
+    (fp_text reference "" (at 0 0) (layer "F.SilkS")
+      (effects (font (size 1.27 1.27) (thickness 0.15)))
+    )
+    (fp_text value "" (at 0 0) (layer "F.SilkS")
+      (effects (font (size 1.27 1.27) (thickness 0.15)))
+    )
+    (pad "1" thru_hole circle locked (at 0 0) (size 6.4 6.4) (drill 3.2) (layers F&B.Cu *.Mask))
+  )
+  (footprint "MountingHole:MountingHole_3.2mm_M3_Pad" locked (layer "F.Cu")
+    (at 156.2 92.84)
+    (descr "Mounting Hole 3.2mm, M3")
+    (tags "mounting hole 3.2mm m3")
+    (attr exclude_from_pos_files exclude_from_bom)
+    (fp_text reference "REF**" (at 0 -4.2) (layer "F.SilkS") hide
+      (effects (font (size 1 1) (thickness 0.15)))
+    )
+    (fp_text value "MountingHole_3.2mm_M3_Pad" (at 0 4.2) (layer "F.Fab") hide
+      (effects (font (size 1 1) (thickness 0.15)))
+    )
+    (fp_text user "${REFERENCE}" (at 0 0) (layer "F.Fab")
+      (effects (font (size 1 1) (thickness 0.15)))
+    )
+    (fp_circle (center 0 0) (end 3.2 0) (layer "Cmts.User") (width 0.15) (fill none))
+    (fp_circle (center 0 0) (end 3.45 0) (layer "F.CrtYd") (width 0.05) (fill none))
+    (pad "1" thru_hole circle locked (at 0 0) (size 6.4 6.4) (drill 3.2) (layers *.Cu *.Mask))
+  )
   (footprint "Capacitor_SMD:CP_Elec_8x11.9" (layer "F.Cu")
-    (at 185.75 68.5 90)
+    (at 155.5 107.5 -90)
     (descr "SMD capacitor, aluminum electrolytic, Panasonic E12, 8.0x11.9mm")
     (tags "capacitor electrolytic")
@@
     (fp_line (start -3.162278 -1.9) (end -3.162278 -1.1) (layer "F.Fab") (width 0.1))
     (fp_circle (center 0 0) (end 4 0) (layer "F.Fab") (width 0.1) (fill none))
-    (pad "1" smd roundrect (at -3.475 0 90) (size 4.15 1.9) (layers "F.Cu" "F.Paste" "F.Mask") (roundrect_rratio 0.131579)
+    (pad "1" smd roundrect (at -3.475 0 270) (size 4.15 1.9) (layers "F.Cu" "F.Paste" "F.Mask") (roundrect_rratio 0.131579)
       (net 4 "Net-(C3-Pad1)") (pintype "passive"))
-    (pad "2" smd roundrect (at 3.475 0 90) (size 4.15 1.9) (layers "F.Cu" "F.Paste" "F.Mask") (roundrect_rratio 0.131579)
+    (pad "2" smd roundrect (at 3.475 0 270) (size 4.15 1.9) (layers "F.Cu" "F.Paste" "F.Mask") (roundrect_rratio 0.131579)
       (net 2 "GND") (pintype "passive"))
     (model "${KICAD6_3DMODEL_DIR}/Capacitor_SMD.3dshapes/CP_Elec_8x11.9.wrl"
@@
   )
   (footprint "Resistor_SMD:R_0805_2012Metric" (layer "F.Cu")
-    (at 151.5 91.75 -90)
+    (at 130.5 121.75 -90)
     (descr "Resistor SMD 0805 (2012 Metric), square (rectangular) end terminal, IPC_7351 nominal, (Body size source: IPC-SM-782 page 72, https://www.pcb-3d.com/wordpress/wp-content/uploads/ipc-sm-782a_amendment_1_and_2.pdf), generated with kicad-footprint-generator")
     (tags "resistor")
@@
     )
   )
+  (footprint "" locked (layer "F.Cu")
+    (at 109 92.84)
+    (fp_text reference "" (at 0 0) (layer "F.SilkS")
+      (effects (font (size 1.27 1.27) (thickness 0.15)))
+    )
+    (fp_text value "" (at 0 0) (layer "F.SilkS")
+      (effects (font (size 1.27 1.27) (thickness 0.15)))
+    )
+    (pad "1" thru_hole circle locked (at 0 0) (size 6.4 6.4) (drill 3.2) (layers F&B.Cu *.Mask))
+  )
   (footprint "Resistor_SMD:R_0612_1632Metric" (layer "F.Cu")
-    (at 157.75 80.75 -90)
+    (at 137 111.25 -90)
     (descr "Resistor SMD 0612 (1632 Metric), square (rectangular) end terminal, IPC_7351 nominal, (Body size source: https://www.vishay.com/docs/20019/rcwe.pdf), generated with kicad-footprint-generator")
     (tags "resistor")
@@
   )
   (footprint "Resistor_SMD:R_0805_2012Metric" (layer "F.Cu")
-    (at 147.5 95.25 -90)
+    (at 126.5 125.25 -90)
     (descr "Resistor SMD 0805 (2012 Metric), square (rectangular) end terminal, IPC_7351 nominal, (Body size source: IPC-SM-782 page 72, https://www.pcb-3d.com/wordpress/wp-content/uploads/ipc-sm-782a_amendment_1_and_2.pdf), generated with kicad-footprint-generator")
     (tags "resistor")
@@
   )
   (footprint "Capacitor_SMD:CP_Elec_8x10.5" (layer "F.Cu")
-    (at 146 68.95 90)
+    (at 115.75 110.75 -90)
     (descr "SMD capacitor, aluminum electrolytic, Vishay 0810, 8.0x10.5mm, http://www.vishay.com/docs/28395/150crz.pdf")
     (tags "capacitor electrolytic")
@@
     (fp_line (start -3.25 4.25) (end 4.25 4.25) (layer "F.Fab") (width 0.1))
     (fp_circle (center 0 0) (end 4 0) (layer "F.Fab") (width 0.1) (fill none))
-    (pad "1" smd roundrect (at -3.7 0 90) (size 4.4 2.5) (layers "F.Cu" "F.Paste" "F.Mask") (roundrect_rratio 0.1)
+    (pad "1" smd roundrect (at -3.7 0 270) (size 4.4 2.5) (layers "F.Cu" "F.Paste" "F.Mask") (roundrect_rratio 0.1)
       (net 1 "Net-(C2-Pad1)") (pintype "passive"))
-    (pad "2" smd roundrect (at 3.7 0 90) (size 4.4 2.5) (layers "F.Cu" "F.Paste" "F.Mask") (roundrect_rratio 0.1)
+    (pad "2" smd roundrect (at 3.7 0 270) (size 4.4 2.5) (layers "F.Cu" "F.Paste" "F.Mask") (roundrect_rratio 0.1)
       (net 2 "GND") (pintype "passive"))
     (model "${KICAD6_3DMODEL_DIR}/Capacitor_SMD.3dshapes/CP_Elec_8x10.5.wrl"
@@
   )
   (footprint "Package_SON:VSONP-8-1EP_5x6_P1.27mm" (layer "F.Cu")
-    (at 158.385 75.45 90)
+    (at 137.75 105.5 90)
     (descr "SON, 8-Leads, Body 5x6x1mm, Pitch 1.27mm; (see Texas Instruments CSD18531Q5A http://www.ti.com/lit/ds/symlink/csd18531q5a.pdf)")
     (tags "VSONP 1.27")
@@
   )
   (footprint "Capacitor_SMD:CP_Elec_8x10.5" (layer "F.Cu")
-    (at 146 81.45 -90)
+    (at 125 110.8 -90)
     (descr "SMD capacitor, aluminum electrolytic, Vishay 0810, 8.0x10.5mm, http://www.vishay.com/docs/28395/150crz.pdf")
     (tags "capacitor electrolytic")
@@
   )
   (footprint "Capacitor_SMD:CP_Elec_8x11.9" (layer "F.Cu")
-    (at 185.75 80.5 -90)
+    (at 146.5 107.5 -90)
     (descr "SMD capacitor, aluminum electrolytic, Panasonic E12, 8.0x11.9mm")
     (tags "capacitor electrolytic")
@@
     )
   )
+  (gr_rect (start 100 87) (end 165 125) (layer "User.1") (width 0.1) (fill none))
+  (gr_rect locked (start 109 92.84) (end 156.2 119) (layer "User.2") (width 0.15) (fill none))
 )

Commit message: Add 3d model, finish layout pending type-c plug study
Parts:
- added C7: 470nF, Capacitor_SMD:C_0805_2012Metric, F.Cu at (148.5, 117.2)
- added J1: Conn_01x02, TerminalBlock_Phoenix:TerminalBlock_Phoenix_PT-1,5-2-5.0-H_1x02_P5.00mm_Horizontal, B.Cu at (98.7, 107.7)
- added U2: TDS2211P.C, Library:DFN-6_1.6x1.6, F.Cu at (109.2, 105.0)
- added U3: TDS2211P.C, Library:DFN-6_1.6x1.6, F.Cu at (162.2, 107.0)
- D1: value D_Schottky_AKA -> STPS20M100SG
- Q1: value Q_NMOS_SGD -> CSD17311Q5
- moved C5 7.92 mm to (131.8, 118.5)
- moved C6 7.92 mm to (133.8, 118.5)
- moved R2 7.92 mm to (133.8, 122.0)
- moved R4 7.92 mm to (135.8, 118.5)
- moved R5 7.92 mm to (137.8, 118.5)
- moved U1 4.07 mm to (143.2, 117.2)
- moved R1 3.34 mm to (141.8, 121.0)
Routing:
- net Net-(C3-Pad1): track 0.00 -> 35.1 mm, vias 0 -> 2
- net Net-(C1-Pad1): track 0.00 -> 24.4 mm, vias 0 -> 2
- net Net-(Q1-Pad2): track 0.00 -> 14.6 mm, vias 0 -> 2
- net Net-(Q1-Pad1): track 0.00 -> 12.0 mm, vias 0 -> 2
- net Net-(C5-Pad2): track 0.00 -> 10.6 mm
- net GND: track 0.00 -> 6.27 mm, vias 0 -> 5
- net Net-(R1-Pad2): track 0.00 -> 6.17 mm
- net Net-(R4-Pad2): track 0.00 -> 5.33 mm
- net Net-(C6-Pad1): track 0.00 -> 1.64 mm
- net Net-(D1-Pad1): vias 0 -> 48
- added copper zone on B.Cu, net GND
- added copper zone on F.Cu, net GND
- added copper zone on F.Cu, net Net-(C1-Pad1)
- added copper zone on F.Cu, net Net-(C3-Pad1)
- added copper zone on B.Cu, net Net-(D1-Pad1)
- added copper zone on F.Cu, net Net-(D1-Pad1)
- added copper zone on F.Cu, net Net-(Q1-Pad1)
Other:
- board outline added: 72 x 41.8 mm
- board text added: "+ Input"
- board text added: "FRC 639 Vision PSU"
