File: coprocessor-psu.kicad_sch (KiCad schematic)
At the start: 15 parts, among them Q1 Q_NMOS_SGD, U1 LM3488

Commit message: Add 3d model, finish layout pending type-c plug study
Parts:
- added C7: 470nF, Capacitor_SMD:C_0805_2012Metric, symbol Device:C
- added J1: Conn_01x02, TerminalBlock_Phoenix:TerminalBlock_Phoenix_PT-1,5-2-5.0-H_1x02_P5.00mm_Horizontal, symbol Connector_Generic:Conn_01x02
- added J2: Conn_01x02, symbol Connector_Generic:Conn_01x02
- added U2, U3: TDS2211P.C, Library:DFN-6_1.6x1.6, symbol symbol:TDS2211P.C
- C1, C2: MPN (none) -> EEE-FN1E471UV
- C3, C4: MPN (none) -> 35SVPF82M
- C5: MPN (none) -> CGA4J1C0G2A333J125AE
- C6: MPN (none) -> CGA4J3X7R1H474K125AE
- D1: value D_Schottky_AKA -> STPS20M100SG; footprint (none) -> Package_TO_SOT_SMD:TO-263-2; MPN (none) -> STPS20M100SG
- L1: MPN (none) -> XAL1580-532MED
- Q1: value Q_NMOS_SGD -> CSD17311Q5; MPN (none) -> CSD17311Q5
- R3: MPN (none) -> WSL06123L000FEA
- U1: MPN (none) -> LM3488MM
Connections:
- net GND: now also C7.1, J1.1 (Pin_1), J2.2 (Pin_2), U2.1, U2.2, U2.3, U3.1, U3.2, U3.3
- net at C1.1, C2.1, L1.1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: now also C7.2, J1.2 (Pin_2), U2.4, U2.5, U2.6
- net at C3.1, C4.1, D1.2 (K)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: now also J2.1 (Pin_1), U3.4, U3.5, U3.6
Other:
- moved on the sheet: C1, C2, C3, C4, C5, C6, D1, L1, Q1, R1, R2, R3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
